File: hw/analog.sch (KiCad schematic (older format))
At the start: 18 parts, among them J5 Conn_01x03, Q1 STT6N3LLH6, Q2 IKW40N120H3FKSA1, U6 MCP1407-E/SN, U7 SCS-200LD

Commit message: Hardware fix.
Added pull-down resistor on PWM output of the MCU so the charge pump
gate does not get charged when the PWM pin is floating.
Parts:
- added R11: 10M, Resistor_SMD:R_0603_1608Metric, symbol Device:R_Small
Connections:
- net CHARGE_PWM: now also R11.1
- net GND: now also R11.2
Other:
- note added: "If the gate if floating when not driven by the MCU\n(for example when reprogramming the device), it\nmay charge overtime...\nA high impedance pull-down may help."
Changed lines of the file:
@@
 Wire Wire Line
 	1000 1100 1000 1300
-Wire Wire Line
-	1700 3400 1400 3400
 Text Notes 4000 4450 0    50   ~ 0
 Bridge to adapt voltage to ADC input range.\nAlso acts a bleeding resistors for safety.
@@
 Wire Wire Line
 	7450 4200 8300 4200
+$Comp
+L Device:R_Small R?
+U 1 1 5DCDDCD3
+P 1550 3600
+AR Path="/5DCDDCD3" Ref="R?"  Part="1"
+AR Path="/5D9F87D8/5DCDDCD3" Ref="R11"  Part="1"
+F 0 "R11" H 1609 3646 50  0000 L CNN
+F 1 "10M" H 1609 3555 50  0000 L CNN
+F 2 "Resistor_SMD:R_0603_1608Metric" H 1550 3600 50  0001 C CNN
+F 3 "~" H 1550 3600 50  0001 C CNN
+F 4 "Multicomp" H -3550 500 50  0001 C CNN "Manufacturer"
+F 5 "MCWR06W1005FTL" H -3550 500 50  0001 C CNN "ManufacturerRef"
+F 6 "0.0046" H -3550 500 50  0001 C CNN "Price"
+F 7 "Farnell" H -3550 500 50  0001 C CNN "Vendor"
+F 8 "2447232" H -3550 500 50  0001 C CNN "VendorRef"
+	1    1550 3600
+	1    0    0    -1
+$EndComp
+$Comp
+L power:GND #PWR?
+U 1 1 5DCDDD42
+P 1550 3800
+AR Path="/5DCDDD42" Ref="#PWR?"  Part="1"
+AR Path="/5D9F87D8/5DCDDD42" Ref="#PWR0121"  Part="1"
+F 0 "#PWR0121" H 1550 3550 50  0001 C CNN
+F 1 "GND" H 1555 3627 50  0000 C CNN
+F 2 "" H 1550 3800 50  0001 C CNN
+F 3 "" H 1550 3800 50  0001 C CNN
+	1    1550 3800
+	1    0    0    -1
+$EndComp
+Wire Wire Line
+	1550 3800 1550 3700
+Wire Wire Line
+	1400 3400 1550 3400
+Wire Wire Line
+	1550 3500 1550 3400
+Connection ~ 1550 3400
+Wire Wire Line
+	1550 3400 1700 3400
+Text Notes 750  4450 0    50   ~ 0
+If the gate if floating when not driven by the MCU\n(for example when reprogramming the device), it\nmay charge overtime...\nA high impedance pull-down may help.
 $EndSCHEMATC

Commit message: Fixed IGBT footprint.
Parts:
- Q2: footprint mykicadlibs:TO-247-3_Horizontal_TabUp_NoTabDrill -> mykicadlibs:TO-247-3_Horizontal_TabDown_NoTabDrill
Changed lines of the file:
@@
 F 0 "Q2" H 10091 4246 50  0000 L CNN
 F 1 "IKW40N120H3FKSA1" H 10091 4155 50  0000 L CNN
-F 2 "mykicadlibs:TO-247-3_Horizontal_TabUp_NoTabDrill" H 10100 4300 50  0001 C CNN
+F 2 "mykicadlibs:TO-247-3_Horizontal_TabDown_NoTabDrill" H 10100 4300 50  0001 C CNN
 F 3 "https://www.infineon.com/dgdl/Infineon-IKW40N120H3-DS-v02_01-EN.pdf?fileId=db3a304325305e6d012591d4832f7032" H 9900 4200 50  0001 C CNN
 F 4 "Infineon" H 9900 4200 50  0001 C CNN "Manufacturer"
