File: hw/emfi.kicad_pcb (KiCad board)
At the start: 2 copper layers, 132.5 x 38 mm, 81 parts, among them J1 USB_B_Micro, J2 Conn_Coaxial, J3 Conn_Coaxial, J4 Conn_01x02, J5 Conn_01x03, J6 Conn_Coaxial, Q1 STT6N3LLH6, Q2 IKW40N120H3FKSA1, U1 STM32F205RETx, U2 FT232RL, U3 MIC2288, U4 LD1117S33TR_SOT223, U5 LD1117S33TR_SOT223, U6 MCP1407-E/SN, U7 SCS-200LD, U8 74LVC1G32

Commit message: Updated PCB and gerber files
Routing:
- net /analog/ANTENNA_B: track 47.1 -> 43.4 mm
- net Net-(U1-Pad8): track 2.66 -> 0.00 mm, vias 1 -> 0
- net +3V3: track 97.9 -> 96.7 mm
- net GND: vias 301 -> 303
Other:
- rule pad_to_mask_clearance: 0.051 -> 0
