File: hardware/analog.kicad_sch (KiCad schematic)
At the start: 19 parts, among them J5 Conn_01x03, Q1 STT6N3LLH6, Q2 IKW40N120H3FKSA1, U6 MCP1407-E/SN, U7 SCS-200LD

Commit message: Uploading contribution of Sven Freud to replace Current Sense Transformer
Parts:
- removed U7: SCS-200LD, mykicadlibs:SCS-200L, symbol mylib:SCS-200LD
- added J8: Measurement connector, Connector_PinSocket_2.54mm:PinSocket_1x02_P2.54mm_Vertical, symbol Connector_Generic:Conn_01x02
- added T1: CST2010, Transformer_SMD:Transformer_Coilcraft_CST2010, symbol Transformer:CST2010
Connections:
- net GND: now also J8.2 (Pin_2), T1.2
- net SENSE: now also J8.1 (Pin_1)
- net at C18.2: now also T1.4
- net at Q1.1, Q1.2, Q1.5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: now also T1.11
- net at J5.2 (Pin_2): now also T1.12
