File: hardware/emfi.kicad_sch (KiCad schematic)
At the start: 10 parts, among them J1 USB_B_Micro, J2 Conn_Coaxial, J3 Conn_Coaxial, J6 Conn_Coaxial, U8 74LVC1G32

Commit message: Uploading contribution of Sven Freud to replace Current Sense Transformer
Parts:
- added J7: Conn_01x02, Connector_PinHeader_2.54mm:PinHeader_1x02_P2.54mm_Vertical, symbol Connector_Generic:Conn_01x02
Connections:
- net +3V3: now also J7.1 (Pin_1)
- net GND: now also J7.2 (Pin_2)
Other:
- note added: "PWR connector for external access"
