File: hardware/emfi.kicad_pcb (KiCad board)
At the start: 2 copper layers, 132.5 x 38 mm, 81 parts, among them J1 USB_B_Micro, J2 Conn_Coaxial, J3 Conn_Coaxial, J4 Conn_01x02, J5 Conn_01x03, J6 Conn_Coaxial, Q1 STT6N3LLH6, Q2 IKW40N120H3FKSA1, U1 STM32F205RETx, U2 FT232RL, U3 MIC2288, U4 LD1117S33TR_SOT223, U5 LD1117S33TR_SOT223, U6 MCP1407-E/SN, U7 SCS-200LD, U8 74LVC1G32

Commit message: Uploading contribution of Sven Freud to replace Current Sense Transformer
Parts:
- removed U7: SCS-200LD, mykicadlibs:SCS-200L
- added J7: Conn_01x02, Connector_PinHeader_2.54mm:PinHeader_1x02_P2.54mm_Vertical, F.Cu at (55.3, 60.0)
- added J8: Measurement connector, Connector_PinSocket_2.54mm:PinSocket_1x02_P2.54mm_Vertical, F.Cu at (87.9, 62.5)
- added T1: CST2010, Transformer_SMD:Transformer_Coilcraft_CST2010, B.Cu at (90.9, 49.3)
- moved LOGO1 15.7 mm to (47.8, 46.9)
- moved R2 0.50 mm to (90.5, 58.5)
- moved R3 0.50 mm to (87.0, 58.5)
Connections:
- net /analog/CHARGE_PWM renamed /mcu/TIM1_CH1
- net /mcu/ADC renamed /mcu/ADC123_IN0
- net /mcu/RX renamed /ft232/TX
- J1 pad 4: Net-(J1-Pad4) -> unconnected-(J1-ID-Pad4)
- U1 pad 10: Net-(U1-Pad10) -> unconnected-(U1-PC2-Pad10)
- U1 pad 11: Net-(U1-Pad11) -> unconnected-(U1-PC3-Pad11)
- U1 pad 15: Net-(U1-Pad15) -> unconnected-(U1-PA1-Pad15)
- U1 pad 16: Net-(U1-Pad16) -> unconnected-(U1-PA2-Pad16)
- U1 pad 17: Net-(U1-Pad17) -> unconnected-(U1-PA3-Pad17)
- U1 pad 20: Net-(U1-Pad20) -> unconnected-(U1-PA4-Pad20)
- U1 pad 21: Net-(U1-Pad21) -> unconnected-(U1-PA5-Pad21)
- U1 pad 22: Net-(U1-Pad22) -> unconnected-(U1-PA6-Pad22)
- U1 pad 23: Net-(U1-Pad23) -> unconnected-(U1-PA7-Pad23)
- U1 pad 24: Net-(U1-Pad24) -> unconnected-(U1-PC4-Pad24)
- U1 pad 25: Net-(U1-Pad25) -> unconnected-(U1-PC5-Pad25)
- U1 pad 26: Net-(U1-Pad26) -> unconnected-(U1-PB0-Pad26)
- U1 pad 27: Net-(U1-Pad27) -> unconnected-(U1-PB1-Pad27)
- U1 pad 29: Net-(U1-Pad29) -> unconnected-(U1-PB10-Pad29)
- U1 pad 33: Net-(U1-Pad33) -> unconnected-(U1-PB12-Pad33)
- U1 pad 34: Net-(U1-Pad34) -> unconnected-(U1-PB13-Pad34)
- U1 pad 35: Net-(U1-Pad35) -> unconnected-(U1-PB14-Pad35)
- U1 pad 36: Net-(U1-Pad36) -> unconnected-(U1-PB15-Pad36)
- U1 pad 37: Net-(U1-Pad37) -> unconnected-(U1-PC6-Pad37)
- U1 pad 38: Net-(U1-Pad38) -> unconnected-(U1-PC7-Pad38)
- U1 pad 39: Net-(U1-Pad39) -> unconnected-(U1-PC8-Pad39)
- U1 pad 4: Net-(U1-Pad4) -> unconnected-(U1-PC15-Pad4)
- U1 pad 40: Net-(U1-Pad40) -> unconnected-(U1-PC9-Pad40)
- U1 pad 44: Net-(U1-Pad44) -> unconnected-(U1-PA11-Pad44)
- U1 pad 45: Net-(U1-Pad45) -> unconnected-(U1-PA12-Pad45)
- U1 pad 49: Net-(U1-Pad49) -> unconnected-(U1-PA14-Pad49)
- U1 pad 5: Net-(U1-Pad5) -> unconnected-(U1-PH0-Pad5)
- U1 pad 50: Net-(U1-Pad50) -> unconnected-(U1-PA15-Pad50)
- U1 pad 51: Net-(U1-Pad51) -> unconnected-(U1-PC10-Pad51)
- U1 pad 52: Net-(U1-Pad52) -> unconnected-(U1-PC11-Pad52)
- U1 pad 53: Net-(U1-Pad53) -> unconnected-(U1-PC12-Pad53)
- U1 pad 54: Net-(U1-Pad54) -> unconnected-(U1-PD2-Pad54)
- U1 pad 55: Net-(U1-Pad55) -> unconnected-(U1-PB3-Pad55)
- U1 pad 56: Net-(U1-Pad56) -> unconnected-(U1-PB4-Pad56)
- U1 pad 57: Net-(U1-Pad57) -> unconnected-(U1-PB5-Pad57)
- U1 pad 58: Net-(U1-Pad58) -> unconnected-(U1-PB6-Pad58)
- U1 pad 59: Net-(U1-Pad59) -> unconnected-(U1-PB7-Pad59)
- U1 pad 6: Net-(U1-Pad6) -> unconnected-(U1-PH1-Pad6)
- U1 pad 61: Net-(U1-Pad61) -> unconnected-(U1-PB8-Pad61)
- U1 pad 62: Net-(U1-Pad62) -> unconnected-(U1-PB9-Pad62)
- U1 pad 8: Net-(U1-Pad8) -> unconnected-(U1-PC0-Pad8)
- U1 pad 9: Net-(U1-Pad9) -> unconnected-(U1-PC1-Pad9)
- U2 pad 10: Net-(U2-Pad10) -> unconnected-(U2-DCD-Pad10)
- U2 pad 11: Net-(U2-Pad11) -> unconnected-(U2-CTS-Pad11)
- U2 pad 12: Net-(U2-Pad12) -> unconnected-(U2-CBUS4-Pad12)
- U2 pad 13: Net-(U2-Pad13) -> unconnected-(U2-CBUS2-Pad13)
- U2 pad 14: Net-(U2-Pad14) -> unconnected-(U2-CBUS3-Pad14)
- U2 pad 19: Net-(U2-Pad19) -> unconnected-(U2-~{RESET}-Pad19)
- U2 pad 2: Net-(U2-Pad2) -> unconnected-(U2-DTR-Pad2)
- U2 pad 22: Net-(U2-Pad22) -> unconnected-(U2-CBUS1-Pad22)
- U2 pad 23: Net-(U2-Pad23) -> unconnected-(U2-CBUS0-Pad23)
- U2 pad 27: Net-(U2-Pad27) -> unconnected-(U2-OSCI-Pad27)
- U2 pad 28: Net-(U2-Pad28) -> unconnected-(U2-OSCO-Pad28)
- U2 pad 3: Net-(U2-Pad3) -> unconnected-(U2-RTS-Pad3)
- U2 pad 6: Net-(U2-Pad6) -> unconnected-(U2-RI-Pad6)
- U2 pad 9: Net-(U2-Pad9) -> unconnected-(U2-DCR-Pad9)
- U6 pad 3: Net-(U6-Pad3) -> unconnected-(U6-NC-Pad3)
Routing:
- net Net-(C18-Pad2): track 4.72 -> 14.5 mm, vias 0 -> 1
- net Net-(J5-Pin_2): track 13.0 -> 19.9 mm, vias 0 -> 1
- net Net-(Q1-Pad1): track 18.4 -> 12.2 mm, vias 0 -> 1
- net +3V3: track 96.7 -> 102.6 mm
- net GND: track 159.8 -> 155.5 mm, vias 303 -> 302
- net /mcu/ADC123_IN0: track 27.3 -> 30.4 mm
- net +3V3A: track 39.8 -> 40.5 mm, vias 1 -> 2
Other:
- board text added: "+"
- board text added: "-"
- board text added: "3V3"
- board text added: "BOOT0"
- board text added: "GND"
- board text added: "SiliconToaster v0.2_mod_SF"
- board text removed: "SiliconToaster v0.2"

Commit message: Slickscreen update
Other:
- board text added: "SiliconToaster v0.3"
- board text removed: "SiliconToaster v0.2_mod_SF"
Changed lines of the file:
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@@
 		)
 	)
-	(gr_text "SiliconToaster v0.2_mod_SF"
-		(at 60.5 31.5 0)
+	(gr_text "SiliconToaster v0.3"
+		(at 45 31.5 0)
 		(layer "F.SilkS")
 		(effects
@@
 				(thickness 0.3)
 			)
+			(justify left)
 		)
 	)
